Commit message: Removed typos

File: models/pioneer.xacro (robot description, xacro)
@@ -5,4 +5,4 @@
        xmlns:xacro="http://ros.org/wiki/xacro"
 name="pioneer3at">
-<include filename="$(find p2os_urdf)/urdf/pioneer.xacro"/>
+<xacro:include filename="$(find p2os_urdf)/defs/pioneer3at.xacro"/>
 </robot>

File: models/pioneer1.xacro (robot description, xacro)
@@ -5,5 +5,5 @@
        xmlns:xacro="http://ros.org/wiki/xacro"
 name="pioneer3at">
-<include filename="$(find p2os_urdf)/urdf/pioneer.xacro"/>
+<xacro:include filename="$(find pioneer_outdoor)/models/pioneer.xacro"/>
 <link name="laser"/>
 <link name="gps"/>

File: models/pioneer2.xacro (robot description, xacro)
@@ -5,6 +5,8 @@
        xmlns:xacro="http://ros.org/wiki/xacro"
 name="pioneer3at">
-<include filename="$(find p2os_urdf)/urdf/pioneer.xacro"/>
+<xacro:include filename="$(find p2os_urdf)/urdf/pioneer.xacro"/>
 <link name="laser"/>
+<link name="gps"/>
+<link name="imu"/>
 <joint name="laser_joint" type="fixed">
 		<origin xyz="0.15 0 0.3" rpy="0 0 0"/>
@@ -12,3 +14,13 @@
 		<child link="laser"/>
 </joint>
+<joint name="imu_joint" type="fixed">
+		<origin xyz="0.15 0 0.3" rpy="0 0 0"/>
+		<parent link="base_link"/>
+		<child link="imu"/>
+</joint>
+<joint name="gps_joint" type="fixed">
+		<origin xyz="0.0 0 47" rpy="0 0 0"/>
+		<parent link="base_link"/>
+		<child link="gps"/>
+</joint>
 </robot>

File: models/pioneer3.xacro (robot description, xacro)
@@ -5,5 +5,5 @@
        xmlns:xacro="http://ros.org/wiki/xacro"
 name="pioneer3at">
-<include filename="$(find p2os_urdf)/urdf/pioneer.xacro"/>
+<include filename="$(find pioneer_outdoor)/models/pioneer.xacro"/>
 <link name="laser"/>
 <link name="gps"/>
